Commit message: update gravity compensation through roughly urdf guessing and dynamic identification needed to test

File: configs/models/X5_camera.urdf (robot description, URDF)
Before this commit: robot X5, 8 links, 7 joints
Links:
- link eef_link: mass 0.072 -> None
- link link6: mass 0.581000 -> 0.653
